File: hardware/warp-energy-manager-v2.kicad_sch (KiCad schematic)
At the start: 113 parts, among them J101 Boot, J102 DM3CS, P101 CON-SENSOR2, P102 SG-Ready, P103 L+N, P104 OUT, P105 INPUT, P110 MODBUS, P111 Debug, Q101 2N7002P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

Commit message: add logos
Parts:
- R104, R105, R115, R116: value 2k2 -> 4k7
- R111, R119: value 1k -> 2k2
- R112, R117, R120, R121: value 680 -> 1k
Connections:
- net RELAY0: now also Q102.G, R110.2, U101.23 (P1.3_IHO); no longer Q107.G, R113.2, U101.24 (P1.2_IHO)
- net RELAY1: now also Q107.G, R113.2, U101.24 (P1.2_IHO); no longer Q102.G, R110.2, U101.23 (P1.3_IHO)
- net SG-OUT-0: now also Q101.G, R102.2, U101.21 (P1.5_IHO); no longer Q103.G, R118.2, U101.22 (P1.4_IHO)
- net SG-OUT-1: now also Q103.G, R118.2, U101.22 (P1.4_IHO); no longer Q101.G, R102.2, U101.21 (P1.5_IHO)
Other:
- note added: "ca 70mW per input"
Changed lines of the file:
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@@
 		)
 	)
+	(text "ca 70mW per input"
+		(exclude_from_sim no)
+		(at 194.31 263.525 0)
+		(effects
+			(font
+				(size 0.9906 0.9906)
+			)
+			(justify right bottom)
+		)
+	)
 	(text "SPI Slave/CH0\nP0.13 : USIC0_CH0-DX2F : SEL\nP0.14 : USIC0_CH0-DX1A : CLK\nP0.15 : USIC0_CH0-DX0B : MOSI\nP2.0 : USIC0_CH0-DOUT0 : MISO"
 		(exclude_from_sim no)
@@
 		)
 	)
-	(global_label "SG-OUT-1"
+	(global_label "SG-OUT-0"
 		(shape input)
 		(at 250.19 77.47 0)
@@
 		)
 	)
-	(global_label "RELAY1"
+	(global_label "RELAY0"
 		(shape output)
 		(at 129.54 81.28 180)
@@
 		)
 	)
-	(global_label "SG-OUT-0"
+	(global_label "SG-OUT-1"
 		(shape output)
 		(at 129.54 83.82 180)
@@
 		)
 	)
-	(global_label "RELAY0"
+	(global_label "RELAY1"
 		(shape output)
 		(at 129.54 78.74 180)
@@
 		)
 	)
-	(global_label "SG-OUT-1"
+	(global_label "SG-OUT-0"
 		(shape output)
 		(at 129.54 86.36 180)
@@
 		)
 	)
-	(global_label "SG-OUT-0"
+	(global_label "SG-OUT-1"
 		(shape input)
 		(at 250.19 38.1 0)
@@
 		)
 	)
-	(global_label "RELAY0"
+	(global_label "RELAY1"
 		(shape input)
 		(at 313.69 45.72 0)
@@
 		)
 	)
-	(global_label "RELAY1"
+	(global_label "RELAY0"
 		(shape input)
 		(at 313.69 95.25 0)
@@
 			)
 		)
-		(property "Value" "1k"
+		(property "Value" "2k2"
 			(at 214.63 179.07 90)
 			(effects
@@
 			)
 		)
-		(property "Value" "680"
+		(property "Value" "1k"
 			(at 214.63 184.15 90)
 			(effects
@@
 			)
 		)
-		(property "Value" "680"
+		(property "Value" "1k"
 			(at 214.63 191.77 90)
 			(effects
@@
 			)
 		)
-		(property "Value" "2k2"
+		(property "Value" "4k7"
 			(at 185.42 199.39 90)
 			(effects
@@
 			)
 		)
-		(property "Value" "2k2"
+		(property "Value" "4k7"
 			(at 180.34 199.39 90)
 			(effects
@@
 			)
 		)
-		(property "Value" "2k2"
+		(property "Value" "4k7"
 			(at 180.34 245.11 90)
 			(effects
@@
 			)
 		)
-		(property "Value" "1k"
+		(property "Value" "2k2"
 			(at 214.63 224.79 90)
 			(effects
@@
 			)
 		)
-		(property "Value" "2k2"
+		(property "Value" "4k7"
 			(at 185.42 245.11 90)
 			(effects
@@
 			)
 		)
-		(property "Value" "680"
+		(property "Value" "1k"
 			(at 214.63 229.87 90)
 			(effects
@@
 			)
 		)
-		(property "Value" "680"
+		(property "Value" "1k"
 			(at 214.63 237.49 90)
 			(effects
